Commit message: change urdf to xacro for scalability and abstraction

File: my_robot_description/urdf/arm.xacro (robot description, xacro)
@@ -1,10 +1,4 @@
 <?xml version="1.0"?>
-<robot name="my_robot">
-    <material name="grey">
-        <color rgba="0.5 0.5 0.5 1.0" />
-    </material>
-    <material name="blue">
-        <color rgba="0.0 0.0 0.5 1.0" />
-    </material>
+<robot xmlns:xacro="http://www.ros.org/wiki/xacro">
     <link name="base_link">
         <visual>

Commit message: add collision tag

File: my_robot_description/urdf/arm.xacro (robot description, xacro)
@@ -9,4 +9,10 @@
             <material name="grey" />
         </visual>
+        <collision>
+            <geometry>
+                <box size="0.4 0.4 0.1" />
+            </geometry>
+            <origin xyz="0 0 0.05" rpy="0 0 0" />
+        </collision>
     </link>
     <link name="shoulder_link">
@@ -18,4 +24,10 @@
             <material name="blue" />
         </visual>
+        <collision>
+            <geometry>
+                <box size="0.2 0.2 0.5" />
+            </geometry>
+            <origin xyz="0 0 0.25" rpy="0 0 0" />
+        </collision>
     </link>
     <link name="arm_link">
@@ -27,4 +39,10 @@
             <material name="grey" />
         </visual>
+        <collision>
+            <geometry>
+                <box size="0.1 0.1 0.6" />
+            </geometry>
+            <origin xyz="0 0 0.3" rpy="0 0 0" />
+        </collision>
     </link>
     <link name="elbow_link">
@@ -36,4 +54,10 @@
             <material name="blue" />
         </visual>
+        <collision>
+            <geometry>
+                <box size="0.1 0.1 0.1" />
+            </geometry>
+            <origin xyz="0 0 0.05" rpy="0 0 0" />
+        </collision>
     </link>
     <link name="forearm_link">
@@ -45,4 +69,10 @@
             <material name="grey" />
         </visual>
+        <collision>
+            <geometry>
+                <box size="0.1 0.1 0.5" />
+            </geometry>
+            <origin xyz="0 0 0.25" rpy="0 0 0" />
+        </collision>
     </link>
     <link name="wrist_link">
@@ -54,4 +84,10 @@
             <material name="blue" />
         </visual>
+        <collision>
+            <geometry>
+                <box size="0.1 0.1 0.05" />
+            </geometry>
+            <origin xyz="0 0 0.025" rpy="0 0 0" />
+        </collision>
     </link>
     <link name="hand_link">
@@ -63,4 +99,10 @@
             <material name="grey" />
         </visual>
+        <collision>
+            <geometry>
+                <box size="0.1 0.1 0.02" />
+            </geometry>
+            <origin xyz="0 0 0.01" rpy="0 0 0" />
+        </collision>
     </link>
     <link name="tool_link" />
